Commit message: check aliengo black.usd

File: assets/URDF/aliengo_black.urdf (robot description, URDF)
Before this commit: robot aliengo, 31 links, 30 joints
Links:
- link FL_calf: geometry collision box size=0.25 0.0208 0.016; visual mesh filename=/home/robotac22/RL_Dog/assets/MESHES/calf.dae scale=1 1 1
- link FL_hip: geometry collision cylinder length=0.0418 radius=0.046; visual mesh filename=/home/robotac22/RL_Dog/assets/MESHES/hip.dae scale=1 1 1
- link FL_thigh: geometry collision box size=0.25 0.0374 0.043; visual mesh filename=/home/robotac22/RL_Dog/assets/MESHES/thigh.dae scale=1 1 1
- link FR_calf: geometry collision box size=0.25 0.0208 0.016; visual mesh filename=/home/robotac22/RL_Dog/assets/MESHES/calf.dae scale=1 1 1
- link FR_hip: geometry collision cylinder length=0.0418 radius=0.046; visual mesh filename=/home/robotac22/RL_Dog/assets/MESHES/hip.dae scale=1 1 1
- link FR_thigh: geometry collision box size=0.25 0.0374 0.043; visual mesh filename=/home/robotac22/RL_Dog/assets/MESHES/thigh_mirror.dae scale=1 1 1
- link RL_calf: geometry collision box size=0.25 0.0208 0.016; visual mesh filename=/home/robotac22/RL_Dog/assets/MESHES/calf.dae scale=1 1 1
- link RL_hip: geometry collision cylinder length=0.0418 radius=0.046; visual mesh filename=/home/robotac22/RL_Dog/assets/MESHES/hip.dae scale=1 1 1
- link RL_thigh: geometry collision box size=0.25 0.0374 0.043; visual mesh filename=/home/robotac22/RL_Dog/assets/MESHES/thigh.dae scale=1 1 1
- link RR_calf: geometry collision box size=0.25 0.0208 0.016; visual mesh filename=/home/robotac22/RL_Dog/assets/MESHES/calf.dae scale=1 1 1
- link RR_hip: geometry collision cylinder length=0.0418 radius=0.046; visual mesh filename=/home/robotac22/RL_Dog/assets/MESHES/hip.dae scale=1 1 1
- link RR_thigh: geometry collision box size=0.25 0.0374 0.043; visual mesh filename=/home/robotac22/RL_Dog/assets/MESHES/thigh_mirror.dae scale=1 1 1
- link trunk: geometry collision box size=0.647 0.15 0.112; visual mesh filename=/home/robotac22/RL_Dog/assets/MESHES/trunk.dae scale=1 1 1

File: assets/URDF/aliengo_color.urdf (robot description, URDF)
Before this commit: robot aliengo, 31 links, 30 joints
Links:
- link FL_calf: geometry collision box size=0.25 0.0208 0.016; visual mesh filename=/home/robotac22/RL_Dog/assets/MESHES/calf.dae scale=1 1 1
- link FL_hip: geometry collision cylinder length=0.0418 radius=0.046; visual mesh filename=/home/robotac22/RL_Dog/assets/MESHES/hip.dae scale=1 1 1
- link FL_thigh: geometry collision box size=0.25 0.0374 0.043; visual mesh filename=/home/robotac22/RL_Dog/assets/MESHES/thigh.dae scale=1 1 1
- link FR_calf: geometry collision box size=0.25 0.0208 0.016; visual mesh filename=/home/robotac22/RL_Dog/assets/MESHES/calf.dae scale=1 1 1
- link FR_hip: geometry collision cylinder length=0.0418 radius=0.046; visual mesh filename=/home/robotac22/RL_Dog/assets/MESHES/hip.dae scale=1 1 1
- link FR_thigh: geometry collision box size=0.25 0.0374 0.043; visual mesh filename=/home/robotac22/RL_Dog/assets/MESHES/thigh_mirror.dae scale=1 1 1
- link RL_calf: geometry collision box size=0.25 0.0208 0.016; visual mesh filename=/home/robotac22/RL_Dog/assets/MESHES/calf.dae scale=1 1 1
- link RL_hip: geometry collision cylinder length=0.0418 radius=0.046; visual mesh filename=/home/robotac22/RL_Dog/assets/MESHES/hip.dae scale=1 1 1
- link RL_thigh: geometry collision box size=0.25 0.0374 0.043; visual mesh filename=/home/robotac22/RL_Dog/assets/MESHES/thigh.dae scale=1 1 1
- link RR_calf: geometry collision box size=0.25 0.0208 0.016; visual mesh filename=/home/robotac22/RL_Dog/assets/MESHES/calf.dae scale=1 1 1
- link RR_hip: geometry collision cylinder length=0.0418 radius=0.046; visual mesh filename=/home/robotac22/RL_Dog/assets/MESHES/hip.dae scale=1 1 1
- link RR_thigh: geometry collision box size=0.25 0.0374 0.043; visual mesh filename=/home/robotac22/RL_Dog/assets/MESHES/thigh_mirror.dae scale=1 1 1
- link trunk: geometry collision box size=0.647 0.15 0.112; visual mesh filename=/home/robotac22/RL_Dog/assets/MESHES/trunk.dae scale=1 1 1

Commit message: USD has now meshes correctly (vP proven). DDPG and Safety not showing USD, Stilll problem!

File: assets/URDF/aliengo_black.urdf (robot description, URDF)
Before this commit: robot aliengo, 31 links, 30 joints
Links:
- link FL_calf: geometry collision box size=0.25 0.0208 0.016; visual mesh filename=/home/user/Documents/GitHub/RL_Dog/assets/MESHES/calf.dae scale=1 1 1
- link FL_hip: geometry collision cylinder length=0.0418 radius=0.046; visual mesh filename=/home/user/Documents/GitHub/RL_Dog/assets/MESHES/hip.dae scale=1 1 1
- link FL_thigh: geometry collision box size=0.25 0.0374 0.043; visual mesh filename=/home/user/Documents/GitHub/RL_Dog/assets/MESHES/thigh.dae scale=1 1 1
- link FR_calf: geometry collision box size=0.25 0.0208 0.016; visual mesh filename=/home/user/Documents/GitHub/RL_Dog/assets/MESHES/calf.dae scale=1 1 1
- link FR_hip: geometry collision cylinder length=0.0418 radius=0.046; visual mesh filename=/home/user/Documents/GitHub/RL_Dog/assets/MESHES/hip.dae scale=1 1 1
- link FR_thigh: geometry collision box size=0.25 0.0374 0.043; visual mesh filename=/home/user/Documents/GitHub/RL_Dog/assets/MESHES/thigh_mirr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 scale=1 1 1
- link RL_calf: geometry collision box size=0.25 0.0208 0.016; visual mesh filename=/home/user/Documents/GitHub/RL_Dog/assets/MESHES/calf.dae scale=1 1 1
- link RL_hip: geometry collision cylinder length=0.0418 radius=0.046; visual mesh filename=/home/user/Documents/GitHub/RL_Dog/assets/MESHES/hip.dae scale=1 1 1
- link RL_thigh: geometry collision box size=0.25 0.0374 0.043; visual mesh filename=/home/user/Documents/GitHub/RL_Dog/assets/MESHES/thigh.dae scale=1 1 1
- link RR_calf: geometry collision box size=0.25 0.0208 0.016; visual mesh filename=/home/user/Documents/GitHub/RL_Dog/assets/MESHES/calf.dae scale=1 1 1
- link RR_hip: geometry collision cylinder length=0.0418 radius=0.046; visual mesh filename=/home/user/Documents/GitHub/RL_Dog/assets/MESHES/hip.dae scale=1 1 1
- link RR_thigh: geometry collision box size=0.25 0.0374 0.043; visual mesh filename=/home/user/Documents/GitHub/RL_Dog/assets/MESHES/thigh_mirr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 scale=1 1 1
- link trunk: geometry collision box size=0.647 0.15 0.112; visual mesh filename=/home/user/Documents/GitHub/RL_Dog/assets/MESHES/trunk.dae scale=1 1 1
